File: bluepill-expansion.sch (KiCad schematic (older format))
At the start: 37 parts, among them J1 SENSE_A, J10 ENCODERS, J11 LS2, J12 I/O 3V3, J13 DIGITAL_PWR, J2 SENSE_B, J3 POWER_DC, J4 MOTDC1, J5 MOTDC2, J6 I2C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

Commit message: update PCB
Parts:
- added C7: 0.1uF, Capacitor_THT:C_Disc_D7.5mm_W2.5mm_P5.00mm, symbol Device:C
- added C8: 100uF, Capacitor_THT:CP_Radial_D5.0mm_P2.50mm, symbol Device:CP
- C6: value 100uF -> 470uF
- J13: footprint Connector_PinHeader_2.54mm:PinHeader_1x02_P2.54mm_Vertical -> TerminalBlock:TerminalBlock_bornier-2_P5.08mm
Connections:
- net +5V: now also C7.1, C8.1
- net GND: now also C7.2, C8.2
Other:
- moved on the sheet: C5, C6, J1, J13, J2, J3, J6, J7, J8, R1, R2, R5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

Commit message: 3d fixed
Parts:
- J10: footprint TerminalBlock:TerminalBlock_bornier-6_P5.08mm -> miTerminalBlock:TerminalBlock_bornier-6_P5.08mm
- J13, J3, J4, J5: footprint TerminalBlock:TerminalBlock_bornier-2_P5.08mm -> miTerminalBlock:TerminalBlock_bornier-2_P5.08mm
- SW1, SW2: footprint Button_Switch_THT:SW_PUSH_6mm_H8.5mm -> Button_Switch_THT:SW_PUSH_6mm_H7.3mm
- U2: footprint Package_TO_SOT_THT:TO-220-15_P2.54x2.54mm_StaggerOdd_Lead4.58mm_Vertical -> miPackage_TO_SOT_THT:TO-220-15_P2.54x2.54mm_StaggerOdd_Lead4.58mm_Vertical
Changed lines of the file:
@@
 F 0 "U2" H 1450 3300 50  0000 C CNN
 F 1 "L298HN" H 2250 3300 50  0000 C CNN
-F 2 "Package_TO_SOT_THT:TO-220-15_P2.54x2.54mm_StaggerOdd_Lead4.58mm_Vertical" H 1950 2000 50  0001 L CNN
+F 2 "miPackage_TO_SOT_THT:TO-220-15_P2.54x2.54mm_StaggerOdd_Lead4.58mm_Vertical" H 1950 2000 50  0001 L CNN
 F 3 "http://www.st.com/st-web-ui/static/active/en/resource/technical/document/datasheet/CD00000240.pdf" H 2050 2900 50  0001 C CNN
 	1    1900 2650
@@
 F 0 "J3" H 10480 1642 50  0000 L CNN
 F 1 "POWER_DC" H 10480 1551 50  0000 L CNN
-F 2 "TerminalBlock:TerminalBlock_bornier-2_P5.08mm" H 10400 1650 50  0001 C CNN
+F 2 "miTerminalBlock:TerminalBlock_bornier-2_P5.08mm" H 10400 1650 50  0001 C CNN
 F 3 "~" H 10400 1650 50  0001 C CNN
 	1    10400 1650
@@
 F 0 "J4" H 2180 6692 50  0000 L CNN
 F 1 "MOTDC1" H 2180 6601 50  0000 L CNN
-F 2 "TerminalBlock:TerminalBlock_bornier-2_P5.08mm" H 2100 6700 50  0001 C CNN
+F 2 "miTerminalBlock:TerminalBlock_bornier-2_P5.08mm" H 2100 6700 50  0001 C CNN
 F 3 "~" H 2100 6700 50  0001 C CNN
 	1    2100 6700
@@
 F 0 "J5" H 2180 7042 50  0000 L CNN
 F 1 "MOTDC2" H 2180 6951 50  0000 L CNN
-F 2 "TerminalBlock:TerminalBlock_bornier-2_P5.08mm" H 2100 7050 50  0001 C CNN
+F 2 "miTerminalBlock:TerminalBlock_bornier-2_P5.08mm" H 2100 7050 50  0001 C CNN
 F 3 "~" H 2100 7050 50  0001 C CNN
 	1    2100 7050
@@
 F 0 "J10" H 3750 6600 50  0000 C CNN
 F 1 "ENCODERS" H 3750 7300 50  0000 C CNN
-F 2 "TerminalBlock:TerminalBlock_bornier-6_P5.08mm" H 3750 7000 50  0001 C CNN
+F 2 "miTerminalBlock:TerminalBlock_bornier-6_P5.08mm" H 3750 7000 50  0001 C CNN
 F 3 "~" H 3750 7000 50  0001 C CNN
 	1    3750 7000
@@
 F 0 "J13" H 10472 2832 50  0000 R CNN
 F 1 "DIGITAL_PWR" H 10472 2923 50  0000 R CNN
-F 2 "TerminalBlock:TerminalBlock_bornier-2_P5.08mm" H 10500 2950 50  0001 C CNN
+F 2 "miTerminalBlock:TerminalBlock_bornier-2_P5.08mm" H 10500 2950 50  0001 C CNN
 F 3 "~" H 10500 2950 50  0001 C CNN
 	1    10500 2950
@@
 F 0 "SW1" H 2000 5050 50  0000 C CNN
 F 1 "LS1" H 2250 5050 50  0000 C CNN
-F 2 "Button_Switch_THT:SW_PUSH_6mm_H8.5mm" H 2100 5350 50  0001 C CNN
+F 2 "Button_Switch_THT:SW_PUSH_6mm_H7.3mm" H 2100 5350 50  0001 C CNN
 F 3 "~" H 2100 5350 50  0001 C CNN
 	1    2100 5150
@@
 F 0 "SW2" H 4200 5050 50  0000 C CNN
 F 1 "LS2" H 4450 5050 50  0000 C CNN
-F 2 "Button_Switch_THT:SW_PUSH_6mm_H8.5mm" H 4300 5350 50  0001 C CNN
+F 2 "Button_Switch_THT:SW_PUSH_6mm_H7.3mm" H 4300 5350 50  0001 C CNN
 F 3 "~" H 4300 5350 50  0001 C CNN
 	1    4300 5150

Commit message: cambiosEmma
Parts:
- removed C5, C7: 0.1uF, Capacitor_THT:C_Disc_D7.5mm_W2.5mm_P5.00mm, symbol Device:C
- added T1, T2, T3, T4: miTornillo, miTornillo:M3, symbol miTornillo:miTornillo
Connections:
- no-connect marks 8 -> 6
Other:
- moved on the sheet: C6, C8
Changed lines of the file:
@@
 EESchema Schematic File Version 4
-EELAYER 30 0
+LIBS:bluepill-expansion-cache
+EELAYER 29 0
 EELAYER END
 $Descr A4 11693 8268
@@
 $EndDescr
 $Comp
-L bluepill_breakouts:BluePill_STM32F103C U1
-U 1 1 5E5C52D8
-P 6600 3000
-F 0 "U1" H 6625 1527 50  0000 C CNN
-F 1 "BluePill_STM32F103C" H 6625 1436 50  0000 C CNN
-F 2 "BluePill_breakouts:BluePill_STM32F103C" H 6650 1400 50  0001 C CNN
-F 3 "www.rogerclark.net" H 6600 1500 50  0001 C CNN
-	1    6600 3000
-	1    0    0    -1
-$EndComp
-$Comp
 L power:GND #PWR0101
 U 1 1 5E5C9745
@@
 	1    0    0    -1
 $EndComp
-Wire Wire Line
-	9300 1550 9300 1500
-Wire Wire Line
-	9300 1500 9500 1500
-Wire Wire Line
-	9700 1500 9700 1550
-Wire Wire Line
-	9300 1850 9300 1900
-Wire Wire Line
-	9300 1900 9500 1900
-Wire Wire Line
-	9700 1900 9700 1850
-$Comp
-L Device:C C5
-U 1 1 5E74005C
-P 9300 1700
-F 0 "C5" H 9050 1750 50  0000 L CNN
-F 1 "0.1uF" H 8950 1650 50  0000 L CNN
-F 2 "Capacitor_THT:C_Disc_D7.5mm_W2.5mm_P5.00mm" H 9338 1550 50  0001 C CNN
-F 3 "~" H 9300 1700 50  0001 C CNN
-	1    9300 1700
-	1    0    0    -1
-$EndComp
-Wire Wire Line
-	9500 1400 9500 1500
-Connection ~ 9500 1500
-Wire Wire Line
-	9500 1500 9700 1500
 $Comp
 L power:GND #PWR0116
@@
 Wire Wire Line
 	9500 2000 9500 1900
-Connection ~ 9500 1900
-Wire Wire Line
-	9500 1900 9700 1900
-Connection ~ 9700 1500
 Wire Wire Line
 	10200 1750 10100 1750
@@
 	10100 1750 10100 1900
 Wire Wire Line
-	10100 1900 9700 1900
-Connection ~ 9700 1900
-Wire Wire Line
 	10100 1500 10100 1650
 Wire Wire Line
 	10100 1650 10200 1650
-Wire Wire Line
-	9700 1500 10100 1500
 Text GLabel 7700 2600 2    50   Input ~ 0
 PWM4
@@
 Wire Wire Line
 	7700 2300 7500 2300
-NoConn ~ 6550 1100
-NoConn ~ 6650 1100
 $Comp
 L power:+5V #PWR0126
@@
 L Device:CP C6
 U 1 1 5E740E52
-P 9700 1700
-F 0 "C6" H 9818 1746 50  0000 L CNN
-F 1 "470uF" H 9818 1655 50  0000 L CNN
-F 2 "Capacitor_THT:CP_Radial_D5.0mm_P2.50mm" H 9738 1550 50  0001 C CNN
-F 3 "~" H 9700 1700 50  0001 C CNN
-	1    9700 1700
+P 9500 1700
+F 0 "C6" H 9618 1746 50  0000 L CNN
+F 1 "470uF" H 9618 1655 50  0000 L CNN
+F 2 "Capacitor_THT:CP_Radial_D5.0mm_P2.50mm" H 9538 1550 50  0001 C CNN
+F 3 "~" H 9500 1700 50  0001 C CNN
+	1    9500 1700
 	1    0    0    -1
 $EndComp
@@
 CANRX
 $Comp
-L Device:C C7
-U 1 1 5E746727
-P 9300 2900
-F 0 "C7" H 9050 2950 50  0000 L CNN
-F 1 "0.1uF" H 8950 2850 50  0000 L CNN
-F 2 "Capacitor_THT:C_Disc_D7.5mm_W2.5mm_P5.00mm" H 9338 2750 50  0001 C CNN
-F 3 "~" H 9300 2900 50  0001 C CNN
-	1    9300 2900
-	1    0    0    -1
-$EndComp
-$Comp
 L Device:CP C8
 U 1 1 5E746D99
-P 9700 2900
-F 0 "C8" H 9818 2946 50  0000 L CNN
-F 1 "100uF" H 9818 2855 50  0000 L CNN
-F 2 "Capacitor_THT:CP_Radial_D5.0mm_P2.50mm" H 9738 2750 50  0001 C CNN
-F 3 "~" H 9700 2900 50  0001 C CNN
-	1    9700 2900
+P 9500 2900
+F 0 "C8" H 9618 2946 50  0000 L CNN
+F 1 "100uF" H 9618 2855 50  0000 L CNN
+F 2 "Capacitor_THT:CP_Radial_D5.0mm_P2.50mm" H 9538 2750 50  0001 C CNN
+F 3 "~" H 9500 2900 50  0001 C CNN
+	1    9500 2900
 	1    0    0    -1
 $EndComp
@@
 $EndComp
 Wire Wire Line
-	9300 3050 9300 3150
-Wire Wire Line
-	9300 3150 9500 3150
-Wire Wire Line
-	9700 3150 9700 3050
-Wire Wire Line
-	9700 3150 10150 3150
-Wire Wire Line
 	10150 2950 10150 3150
-Connection ~ 9700 3150
-Wire Wire Line
-	10150 2650 9700 2650
-Wire Wire Line
-	9300 2650 9300 2750
 Wire Wire Line
 	10150 2650 10150 2850
+Wire Wire Line
+	9500 2750 9500 2650
+Wire Wire Line
+	9500 3250 9500 3150
+Wire Wire Line
+	9500 2550 9500 2650
+$Comp
+L miTornillo:miTornillo T1
+U 1 1 5E698231
+P 6300 7500
+F 0 "T1" H 6380 7546 50  0000 L CNN
+F 1 "miTornillo" H 6380 7455 50  0000 L CNN
+F 2 "miTornillo:M3" H 6300 7500 50  0001 C CNN
+F 3 "~" H 6300 7500 50  0001 C CNN
+	1    6300 7500
+	1    0    0    -1
+$EndComp
+$Comp
+L miTornillo:miTornillo T3
+U 1 1 5E69B1BA
+P 5750 7500
+F 0 "T3" H 5830 7546 50  0000 L CNN
+F 1 "miTornillo" H 5830 7455 50  0000 L CNN
+F 2 "miTornillo:M3" H 5750 7500 50  0001 C CNN
+F 3 "~" H 5750 7500 50  0001 C CNN
+	1    5750 7500
+	1    0    0    -1
+$EndComp
+$Comp
+L miTornillo:miTornillo T4
+U 1 1 5E6A8329
+P 6300 7300
+F 0 "T4" H 6380 7346 50  0000 L CNN
+F 1 "miTornillo" H 6380 7255 50  0000 L CNN
+F 2 "miTornillo:M3" H 6300 7300 50  0001 C CNN
+F 3 "~" H 6300 7300 50  0001 C CNN
+	1    6300 7300
+	1    0    0    -1
+$EndComp
+$Comp
+L miTornillo:miTornillo T2
+U 1 1 5E6A8333
+P 5750 7300
+F 0 "T2" H 5830 7346 50  0000 L CNN
+F 1 "miTornillo" H 5830 7255 50  0000 L CNN
+F 2 "miTornillo:M3" H 5750 7300 50  0001 C CNN
+F 3 "~" H 5750 7300 50  0001 C CNN
+	1    5750 7300
+	1    0    0    -1
+$EndComp
 Connection ~ 9500 2650
 Wire Wire Line
-	9500 2650 9300 2650
-Wire Wire Line
-	9700 2750 9700 2650
-Connection ~ 9700 2650
-Wire Wire Line
-	9700 2650 9500 2650
-Wire Wire Line
-	9500 3250 9500 3150
+	9500 2650 10150 2650
+Wire Wire Line
+	9500 3150 10150 3150
+Wire Wire Line
+	9500 3050 9500 3150
 Connection ~ 9500 3150
 Wire Wire Line
-	9500 3150 9700 3150
-Wire Wire Line
-	9500 2550 9500 2650
+	9500 1500 10100 1500
+Wire Wire Line
+	9500 1900 10100 1900
+Wire Wire Line
+	9500 1850 9500 1900
+Connection ~ 9500 1900
+Wire Wire Line
+	9500 1400 9500 1500
+Connection ~ 9500 1500
+Wire Wire Line
+	9500 1500 9500 1550
+$Comp
+L bluepill_breakouts:BluePill_STM32F103C U1
+U 1 1 5E5C52D8
+P 6600 3000
+F 0 "U1" H 6625 1527 50  0000 C CNN
+F 1 "BluePill_STM32F103C" H 6625 1436 50  0000 C CNN
+F 2 "BluePill_breakouts:BluePill_STM32F103C" H 6650 1400 50  0001 C CNN
+F 3 "www.rogerclark.net" H 6600 1500 50  0001 C CNN
+	1    6600 3000
+	1    0    0    -1
+$EndComp
 $EndSCHEMATC

Commit message: CAN R 120
Parts:
- added R6, R7: 120, Resistor_THT:R_Axial_DIN0207_L6.3mm_D2.5mm_P2.54mm_Vertical, symbol Device:R
- T1, T2, T3, T4: symbol miTornillo:miTornillo -> bluepill-expansion-rescue:miTornillo-miTornillo
Connections:
- net CANH: now also R6.1, R7.1
- net CANL: now also R6.2, R7.2
Other:
- moved on the sheet: J6, J7, J8, R5, U3
